File: VexLidarBoard.kicad_sch (KiCad schematic)
At the start: 49 parts, among them J1 RJ9, J2 Conn_01x04_Pin, J3 Conn_01x07_Pin, J4 Conn_01x07_Pin, J5 USB_C_Receptacle_USB2.0_14P, SW1 SW_SPST, SW2 SW_SPST, U1 TPS563200, U2 THVD1420D, U3 NCP1117-3.3_SOT223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

Commit message: routing almost done
Parts:
- C10: value 10uF -> 100nF
Changed lines of the file:
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@@
 			)
 		)
-		(property "Value" "10uF"
+		(property "Value" "100nF"
 			(at 237.236 46.99 0)
 			(effects
