File: VexLidarBoard.kicad_pcb (KiCad board)
At the start: 2 copper layers, 49 parts, among them J1 RJ9, J2 Conn_01x04_Pin, J3 Conn_01x07_Pin, J4 Conn_01x07_Pin, J5 USB_C_Receptacle_USB2.0_14P, SW1 SW_SPST, SW2 SW_SPST, U1 TPS563200, U2 THVD1420D, U3 NCP1117-3.3_SOT223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

Commit message: routing almost done
Parts:
- moved C9 57.2 mm to (240.4, 79.6), turned to -45 degrees
- moved C7 57.0 mm to (221.9, 69.8), turned to 135 degrees
- moved D7 51.4 mm to (233.7, 66.8), turned to -90 degrees
- moved R6 49.4 mm to (233.7, 63.0), turned to 90 degrees
- moved C8 43.9 mm to (236.7, 63.2)
- moved R9 38.1 mm to (240.8, 67.7)
- moved R10 34.6 mm to (244.7, 72.6), turned to 90 degrees
- moved R11 34.2 mm to (244.0, 77.0), turned to 180 degrees
- moved D5 18.5 mm to (244.2, 81.7), turned to -90 degrees
- moved D6 17.0 mm to (246.9, 72.0), turned to -90 degrees
- moved J2 0.36 mm to (245.9, 63.9)
- moved C14 0.25 mm to (234.4, 69.7)
- turned D8 to 180 degrees
- turned D9 to 180 degrees
Routing:
- net /RESET: track 0.00 -> 24.3 mm
- net /USB_D-: track 0.00 -> 21.5 mm
- net /USB_D+: track 0.00 -> 18.8 mm
- net GND: track 10.7 -> 20.1 mm, vias 15 -> 19
- net Net-(D2-A): track 0.00 -> 9.34 mm
- net Net-(J5-CC2): track 0.00 -> 7.05 mm
- net Net-(J5-CC1): track 0.00 -> 6.05 mm, vias 0 -> 2
- net Net-(D7-K): track 0.00 -> 1.79 mm
- added copper zone on B.Cu, net GND

Commit message: done layout
Parts:
- moved D9 21.8 mm to (208.7, 89.2), turned to 0 degrees
- moved D8 21.5 mm to (208.7, 87.1), turned to 0 degrees
- moved R8 14.1 mm to (204.8, 89.2), turned to 180 degrees
- moved R7 13.6 mm to (204.8, 87.1), turned to 180 degrees
- moved R6 4.22 mm to (237.6, 64.5)
- moved D7 4.22 mm to (237.6, 68.3)
- moved R5 2.36 mm to (234.4, 67.7)
- moved C8 2.34 mm to (234.4, 63.6)
- moved R4 2.34 mm to (234.4, 65.7)
- moved R10 1.37 mm to (244.2, 71.4)
- moved C10 1.09 mm to (238.3, 71.8), turned to 0 degrees
- moved D6 0.57 mm to (246.4, 72.3)
Routing:
- net /STAT_LED: track 0.00 -> 32.3 mm, vias 0 -> 2
- net /DBG_LED: track 0.00 -> 32.0 mm, vias 0 -> 2
- net /BOOT: track 0.00 -> 21.8 mm
- net /SWDIO: track 0.00 -> 16.8 mm, vias 0 -> 1
- net /RESET: track 24.3 -> 40.1 mm, vias 0 -> 2
- net /SWCLK: track 0.00 -> 14.1 mm, vias 0 -> 1
- net /USB_D+: track 18.8 -> 26.7 mm
- net GND: track 20.1 -> 26.5 mm, vias 19 -> 21
- net +3.3V: track 17.8 -> 21.1 mm, vias 0 -> 2
- net Net-(D9-K): track 0.00 -> 1.81 mm
- net Net-(D8-K): track 0.00 -> 1.79 mm
- net Net-(J5-CC2): track 7.05 -> 7.79 mm

Commit message: done for real
Parts:
- moved U3 1.17 mm to (227.7, 65.0)
- moved C7 1.14 mm to (223.0, 70.0), turned to 180 degrees
Routing:
- net GND: track 26.5 -> 37.9 mm
- net +3.3V: track 21.1 -> 26.9 mm, vias 2 -> 3
- net /BOOT: track 21.8 -> 22.7 mm, vias 0 -> 2
- net /RESET: track 40.1 -> 40.9 mm
Other:
- board outline added: 69.3 x 31.8 mm
